File: projects/pisc_0_0/piscine_0_0.kicad_sch (KiCad schematic)
At the start: 0 parts

Commit message: finished first draft of schematic 70 errors :(
Parts:
- added C1, C5, C6: ~, symbol bt_pisc_0_0:Capacitor_100nF
- added C2, C3: ~, symbol bt_pisc_0_0:Capacitor_12pf
- added C4: ~, symbol bt_pisc_0_0:Capacitor_1uF
- added D1: ~, symbol bt_pisc_0_0:Diode_Red
- added D2: ~, symbol bt_pisc_0_0:Diode_Green
- added GND1, GND2, GND3, GND4, GND5, GND6, GND7, GND8: ~, symbol bt_pisc_0_0:GND
- added J1: ~, symbol bt_pisc_0_0:gpio_left
- added J2: ~, symbol bt_pisc_0_0:gpio_right
- added J3: ~, symbol bt_pisc_0_0:gpio_small
- added R1, R3: ~, symbol bt_pisc_0_0:Resistor_10k
- added R2: ~, symbol bt_pisc_0_0:Resistor_330
- added SW1: ~, symbol bt_pisc_0_0:Switch_Push
- added U1: ATmega328P-A, symbol bt_pisc_0_0:ATmega328P-A
- added VCC1, VCC2, VCC3, VCC4: ~, symbol bt_pisc_0_0:VCC
- added Y1: ~, symbol bt_pisc_0_0:4pin_quartz
Connections:
- new net: U1.18 (AVCC), U1.4 (VCC)
- new net 16MHz: U1.8 (XTAL2/PB7)
- new net A0: U1.23 (PC0)
- new net A1: U1.24 (PC1)
- new net A2: U1.25 (PC2)
- new net A3: U1.26 (PC3)
- new net A4: U1.27 (PC4)
- new net A5: U1.28 (PC5)
- new net A6: U1.19 (ADC6)
- new net A7: U1.22 (ADC7)
- new net D10: U1.14 (PB2)
- new net D2: U1.32 (PD2)
- new net D3: U1.1 (PD3)
- new net D4: U1.2 (PD4)
- new net D5: U1.9 (PD5)
- new net D6: U1.10 (PD6)
- new net D7: U1.11 (PD7)
- new net D8: U1.12 (PB0)
- new net D9: U1.13 (PB1)
- new net DTR: U1.29 (RESET/PC6)
- new net M0SI: U1.15 (PB3)
- new net MIS0: U1.16 (PB4)
- new net RXI: U1.30 (PD0)
- new net SCK: U1.17 (PB5)
- new net TX0: U1.31 (PD1)
Other:
- note added: "Activity"
- note added: "Power"
- note added: "Reset"

Commit message: updated symbols with correct pins
Parts:
- removed C1, C5, C6: ~, symbol bt_pisc_0_0:Capacitor_100nF
- removed C2, C3: ~, symbol bt_pisc_0_0:Capacitor_12pf
- removed C4: ~, symbol bt_pisc_0_0:Capacitor_1uF
- removed D1: ~, symbol bt_pisc_0_0:Diode_Red
- removed D2: ~, symbol bt_pisc_0_0:Diode_Green
- removed GND1, GND2, GND3, GND4, GND5, GND6, GND7, GND8: ~, symbol bt_pisc_0_0:GND
- removed R1, R3: ~, symbol bt_pisc_0_0:Resistor_10k
- removed R2: ~, symbol bt_pisc_0_0:Resistor_330
- removed SW1: ~, symbol bt_pisc_0_0:Switch_Push
- removed VCC1, VCC2, VCC3, VCC4: ~, symbol bt_pisc_0_0:VCC
- added C1, C5, C6: 100nF, symbol bt_pisc_0_0:Capacitor
- added C2, C3: 12pF, symbol bt_pisc_0_0:Capacitor
- added C4: 1uF, symbol bt_pisc_0_0:Capacitor
- added D1: Red, symbol bt_pisc_0_0:Diode
- added D2: Green, symbol bt_pisc_0_0:Diode
- added R1, R3: 10K, symbol bt_pisc_0_0:Resistor
- added R2: 330, symbol bt_pisc_0_0:Resistor
- added SW2: SW_Push, symbol bt_pisc_0_0:Switch_Push
- J3: value ~ -> FTDI
Connections:
- net M0SI is gone; now on net MOSI: U1.15 (PB3)
- net MIS0 is gone; now on net MISO: U1.16 (PB4)
- net 16MHz: now also Y1.3, C3.1
- net A0: now also J2.8
- net A1: now also J2.7
- net A2: now also J2.6
- net A3: now also J2.5
- net D10: now also J2.12
- net D2: now also J1.8
- net D3: now also J1.7
- net D4: now also J1.6
- net D5: now also J1.5
- net D6: now also J1.4
- net D7: now also J1.3
- net D8: now also J1.2
- net D9: now also J1.1
- net DTR: now also J1.10, J2.3, J3.1, R3.2, SW2.2
- net GND: now also J1.9, J2.2, J3.5, J3.6, U1.3 (GND), Y1.2, Y1.4, C1.2, C2.2, C3.2, C4.2, C5.2, C6.2, D2.2, R1.2
- net RXI: now also J1.11, J3.3
- net SCK: now also J2.9, R2.1
- net TX0: now also J1.12, J3.2
- net VCC: now also J2.1, J2.4, J3.4, U1.18 (AVCC), U1.4 (VCC), C4.1, C5.1, D1.1, R3.1
- net at Y1.1: now also U1.7 (XTAL1/PB6), C2.1
- net MISO: now reaches J2.10
- net MOSI: now reaches J2.11
- net at U1.20 (AREF): now also C1.1
- new net: D2.1, R2.2
- new net: C6.1, SW2.1
- new net: D1.2, R1.1

Commit message: added power_flag to schematic for gnd and vcc
edited gpio symbols to use passive pins
edited quartz crystal to use power input pins for 2 and 4
Parts:
- removed J1: ~, symbol bt_pisc_0_0:gpio_left
- removed J2: ~, symbol bt_pisc_0_0:gpio_right
- removed J3: FTDI, symbol bt_pisc_0_0:gpio_small
- added J1, J2: ~, symbol bt_pisc_0_0:gpio_12
- added J3: ~, symbol bt_pisc_0_0:gpio_6
Connections:
- net A0: now also J1.8
- net A1: now also J1.7
- net A2: now also J1.6
- net A3: now also J1.5
- net D10: now also J1.12
- net D2: now also J2.8
- net D3: now also J2.7
- net D4: now also J2.6
- net D5: now also J2.5
- net D6: now also J2.4
- net D7: now also J2.3
- net D8: now also J2.2
- net D9: now also J2.1
- net DTR: now also J1.3, J2.10, J3.1
- net GND: now also J1.2, J2.9, J3.5, J3.6
- net MISO: now also J1.10
- net MOSI: now also J1.11
- net RXI: now also J2.11, J3.3
- net SCK: now also J1.9
- net TX0: now also J2.12, J3.2
- net VCC: now also J1.1, J1.4, J3.4
- net A4: no longer names the net of U1.27 (PC4)
- net A5: no longer names the net of U1.28 (PC5)
- net A6: no longer names the net of U1.19 (ADC6)
- net A7: no longer names the net of U1.22 (ADC7)
- no-connect marks 0 -> 4
