File: projects/pisc_0_0/piscine_0_0.kicad_sch (KiCad schematic)
At the start: 17 parts, among them SW2 SW_Push, U1 ATmega328P-A

Commit message: added through-hole footprints updated symbols with link to their footprints updated schematic symbols adding backups
Connections:
- net GND: now also D2.1; no longer D2.2
- net VCC: now also D1.2; no longer D1.1
- net at R2.2: now also D2.2; no longer D2.1
- net at R1.1: now also D1.1; no longer D1.2

Commit message: Created function but ugly pcb design for arduino mini pcb design is traced with 0 errors updated schematic to include missing gpio footprints
Parts:
- C1, C2, C3, C4, C5, C6, D1, D2, R1, R2, R3: footprint (none) -> Library:0603
- J1, J2: footprint (none) -> Library:12pin_gpio
- J3: footprint (none) -> Library:6pin_gpio
- SW2: footprint (none) -> Library:TS_3225
- U1: footprint (none) -> Library:ATMEGA328P-AU
- Y1: footprint (none) -> Library:crys_osc_smd3225_4
Changed lines of the file:
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@@
 			)
 		)
-		(property "Footprint" ""
+		(property "Footprint" "Library:0603"
 			(at 105.41 53.34 0)
 			(effects
@@
 			)
 		)
-		(property "Footprint" ""
+		(property "Footprint" "Library:0603"
 			(at 156.21 44.45 0)
 			(effects
@@
 			)
 		)
-		(property "Footprint" ""
+		(property "Footprint" "Library:0603"
 			(at 54.61 40.64 0)
 			(effects
@@
 			)
 		)
-		(property "Footprint" ""
+		(property "Footprint" "Library:TS_3225"
 			(at 173.99 40.64 0)
 			(effects
@@
 			)
 		)
-		(property "Footprint" ""
+		(property "Footprint" "Library:0603"
 			(at 153.67 100.33 0)
 			(effects
@@
 			)
 		)
-		(property "Footprint" ""
+		(property "Footprint" "Library:crys_osc_smd3225_4"
 			(at 140.97 119.38 0)
 			(effects
@@
 			)
 		)
-		(property "Footprint" ""
+		(property "Footprint" "Library:0603"
 			(at 158.75 130.81 0)
 			(effects
@@
 			)
 		)
-		(property "Footprint" ""
+		(property "Footprint" "Library:6pin_gpio"
 			(at 256.54 134.62 0)
 			(effects
@@
 			)
 		)
-		(property "Footprint" ""
+		(property "Footprint" "Library:0603"
 			(at 41.91 40.64 0)
 			(effects
@@
 			)
 		)
-		(property "Footprint" ""
+		(property "Footprint" "Library:0603"
 			(at 44.45 85.09 0)
 			(effects
@@
 			)
 		)
-		(property "Footprint" ""
+		(property "Footprint" "Library:0603"
 			(at 114.3 35.56 0)
 			(effects
@@
 			)
 		)
-		(property "Footprint" ""
+		(property "Footprint" "Library:12pin_gpio"
 			(at 231.14 123.19 0)
 			(effects
@@
 			)
 		)
-		(property "Footprint" ""
+		(property "Footprint" "Library:0603"
 			(at 191.77 36.83 0)
 			(effects
@@
 			)
 		)
-		(property "Footprint" ""
+		(property "Footprint" "Library:ATMEGA328P-AU"
 			(at 69.85 128.27 0)
 			(effects
@@
 			)
 		)
-		(property "Footprint" ""
+		(property "Footprint" "Library:0603"
 			(at 64.77 48.26 0)
 			(effects
@@
 			)
 		)
-		(property "Footprint" ""
+		(property "Footprint" "Library:0603"
 			(at 73.66 48.26 0)
 			(effects
@@
 			)
 		)
-		(property "Footprint" ""
+		(property "Footprint" "Library:12pin_gpio"
 			(at 204.47 120.65 0)
 			(effects
